Commit message: Refactor OpenDoge control framework for improved performance and consistency
- Updated control rates to 1000 Hz across various configurations and nodes.
- Enhanced observation structure in `rl_node.cpp` to align with OpenDoge_train, including new scaling factors and input dimensions.
- Revised joint naming conventions in configuration files to match hardware mappings.
- Improved CAN interface setup to support four channels for motor control.
- Adjusted `ros2_control.yaml` to utilize multiple command interfaces (position, velocity, effort, kp, kd) for each joint.
- Updated README and changelog to reflect changes in control architecture and joint configurations.
- Implemented safety measures in `MotorHardware` for fault detection and damping mode activation.
- Removed unnecessary software filtering for IMU and motor outputs, focusing on hardware capabilities.

File: src/opendoge_description/urdf/opendoge_apx.urdf.xacro (robot description, xacro)
@@ -16,5 +16,5 @@
     <origin xyz="0 0 0.05" rpy="0 0 0"/>
   </joint>
-  <!-- Simple 12-DOF leg layout: FL/FR/HL/HR -->
+  <!-- Simple 12-DOF leg layout: FL/FR/RL/RR -->
   <xacro:macro name="leg" params="prefix x y z yaw pitch roll">
     <link name="${prefix}_hip_link"/>
@@ -34,8 +34,8 @@
       <limit lower="-2.0" upper="2.0" effort="50" velocity="10"/>
     </joint>
-    <link name="${prefix}_knee_link"/>
-    <joint name="${prefix}_knee_joint" type="revolute">
+    <link name="${prefix}_calf_link"/>
+    <joint name="${prefix}_calf_joint" type="revolute">
       <parent link="${prefix}_thigh_link"/>
-      <child link="${prefix}_knee_link"/>
+      <child link="${prefix}_calf_link"/>
       <origin xyz="0 0 -0.2" rpy="0 0 0"/>
       <axis xyz="1 0 0"/>
@@ -44,40 +44,51 @@
   </xacro:macro>
   <!-- Front Left -->
-  <xacro:leg prefix="fl" x="0.15" y="0.075" z="0.0" roll="0" pitch="0" yaw="0"/>
+  <xacro:leg prefix="FL" x="0.15" y="0.075" z="0.0" roll="0" pitch="0" yaw="0"/>
   <!-- Front Right -->
-  <xacro:leg prefix="fr" x="0.15" y="-0.075" z="0.0" roll="0" pitch="0" yaw="0"/>
-  <!-- Hind Left -->
-  <xacro:leg prefix="hl" x="-0.15" y="0.075" z="0.0" roll="0" pitch="0" yaw="0"/>
-  <!-- Hind Right -->
-  <xacro:leg prefix="hr" x="-0.15" y="-0.075" z="0.0" roll="0" pitch="0" yaw="0"/>
+  <xacro:leg prefix="FR" x="0.15" y="-0.075" z="0.0" roll="0" pitch="0" yaw="0"/>
+  <!-- Rear Left -->
+  <xacro:leg prefix="RL" x="-0.15" y="0.075" z="0.0" roll="0" pitch="0" yaw="0"/>
+  <!-- Rear Right -->
+  <xacro:leg prefix="RR" x="-0.15" y="-0.075" z="0.0" roll="0" pitch="0" yaw="0"/>
   <!-- ros2_control placeholder: actual hardware mapping defined in YAML -->
   <ros2_control name="OpendogeHardware" type="system">
     <hardware>
       <plugin>motor_control_interface/MotorHardware</plugin>
-      <param name="can_interface">can0</param>
+      <param name="can_interfaces">can0,can1,can2,can3</param>
       <param name="master_id">253</param>
+      <param name="bitrate">1000000</param>
+      <param name="command_timeout_ms">20</param>
+      <param name="state_timeout_ms">20</param>
+      <param name="fault_reaction">damping</param>
     </hardware>
     <!-- Joint list must match controllers.yaml & policy base.yaml -->
-    <xacro:macro name="register_joint" params="joint_name motor_id">
+    <xacro:macro name="register_joint" params="joint_name motor_id can_interface">
       <joint name="${joint_name}">
         <param name="motor_id">${motor_id}</param>
+        <param name="can_interface">${can_interface}</param>
+        <command_interface name="position"/>
+        <command_interface name="velocity"/>
         <command_interface name="effort"/>
+        <command_interface name="kp"/>
+        <command_interface name="kd"/>
         <state_interface name="position"/>
+        <state_interface name="velocity"/>
         <state_interface name="effort"/>
+        <state_interface name="temperature"/>
+        <state_interface name="fault"/>
       </joint>
     </xacro:macro>
-    <!-- Placeholder motor IDs; update to real mapping -->
-    <xacro:register_joint joint_name="fl_hip_joint" motor_id="1"/>
-    <xacro:register_joint joint_name="fl_thigh_joint" motor_id="2"/>
-    <xacro:register_joint joint_name="fl_knee_joint" motor_id="3"/>
-    <xacro:register_joint joint_name="fr_hip_joint" motor_id="4"/>
-    <xacro:register_joint joint_name="fr_thigh_joint" motor_id="5"/>
-    <xacro:register_joint joint_name="fr_knee_joint" motor_id="6"/>
-    <xacro:register_joint joint_name="hl_hip_joint" motor_id="7"/>
-    <xacro:register_joint joint_name="hl_thigh_joint" motor_id="8"/>
-    <xacro:register_joint joint_name="hl_knee_joint" motor_id="9"/>
-    <xacro:register_joint joint_name="hr_hip_joint" motor_id="10"/>
-    <xacro:register_joint joint_name="hr_thigh_joint" motor_id="11"/>
-    <xacro:register_joint joint_name="hr_knee_joint" motor_id="12"/>
+    <xacro:register_joint joint_name="FL_hip_joint" motor_id="1" can_interface="can0"/>
+    <xacro:register_joint joint_name="FL_thigh_joint" motor_id="2" can_interface="can0"/>
+    <xacro:register_joint joint_name="FL_calf_joint" motor_id="3" can_interface="can0"/>
+    <xacro:register_joint joint_name="FR_hip_joint" motor_id="4" can_interface="can1"/>
+    <xacro:register_joint joint_name="FR_thigh_joint" motor_id="5" can_interface="can1"/>
+    <xacro:register_joint joint_name="FR_calf_joint" motor_id="6" can_interface="can1"/>
+    <xacro:register_joint joint_name="RL_hip_joint" motor_id="7" can_interface="can2"/>
+    <xacro:register_joint joint_name="RL_thigh_joint" motor_id="8" can_interface="can2"/>
+    <xacro:register_joint joint_name="RL_calf_joint" motor_id="9" can_interface="can2"/>
+    <xacro:register_joint joint_name="RR_hip_joint" motor_id="10" can_interface="can3"/>
+    <xacro:register_joint joint_name="RR_thigh_joint" motor_id="11" can_interface="can3"/>
+    <xacro:register_joint joint_name="RR_calf_joint" motor_id="12" can_interface="can3"/>
   </ros2_control>
 </robot>
